Commit message: wheels

File: description/robot_core.xacro (robot description, xacro)
@@ -13,6 +13,8 @@
         <color rgba="0 0 0 1" />
     </material>
+    <!--BASE LINK-->
     <link name="base_link">
     </link>
+    <!--CHASSIS LINK-->
     <joint name="chassis_joint" type="fixed">
         <parent link="base_link"/>
@@ -29,3 +31,31 @@
         </visual>
     </link>
+    <!--LEFT WHEEL LINK-->
+    <joint name="left_wheel_joint" type="continuous">
+        <parent link="base_link"/>
+        <child link="left_wheel"/>
+        <origin xyz="0 0.175 0" rpy="-${pi/2} 0 0" />
+        <axis xyz="0 0 1"/>
+    </joint>
+    <link name="left_wheel">
+        <visual>
+            <geometry>
+                <cylinder radius="0.05" length="0.04"/>
+            </geometry>
+            <material name="blue"/>
+        </visual>
+    <!--RIGHT WHEEL LINK-->
+    <joint name="right_wheel_joint" type="continuous">
+        <parent link="base_link"/>
+        <child link="right_wheel"/>
+        <origin xyz="0 -0.175 0" rpy="${pi/2} 0 0" />
+        <axis xyz="0 0 -1"/>
+    </joint>
+    <link name="right_wheel">
+        <visual>
+            <geometry>
+                <cylinder radius="0.05" length="0.04"/>
+            </geometry>
+            <material name="blue"/>
+        </visual>
 </robot>

Commit message: link name

File: description/robot_core.xacro (robot description, xacro)
@@ -45,4 +45,5 @@
             <material name="blue"/>
         </visual>
+    </link>
     <!--RIGHT WHEEL LINK-->
     <joint name="right_wheel_joint" type="continuous">
@@ -59,3 +60,4 @@
             <material name="blue"/>
         </visual>
+    </link>
 </robot>

Commit message: caster

File: description/robot_core.xacro (robot description, xacro)
@@ -61,3 +61,18 @@
         </visual>
     </link>
+    <!--CASTER WHEEL-->
+    <joint name="caster_wheel_joint" type="fixed">
+        <parent link="chassis"/>
+        <child link="caster_wheel"/>
+        <origin xyz="0 -0.175 0" />
+        <axis xyz="0.24 0 0"/>
+    </joint>
+    <link name="caster_wheel">
+        <visual>
+            <geometry>
+                <sphere radius="0.05" />
+            </geometry>
+            <material name="black"/>
+        </visual>
+    </link>
 </robot>

Commit message: caster xyz

File: description/robot_core.xacro (robot description, xacro)
@@ -65,6 +65,5 @@
         <parent link="chassis"/>
         <child link="caster_wheel"/>
-        <origin xyz="0 -0.175 0" />
-        <axis xyz="0.24 0 0"/>
+        <origin xyz="0.24 0 0" />
     </joint>
     <link name="caster_wheel">

Commit message: collision

File: description/robot_core.xacro (robot description, xacro)
@@ -30,4 +30,10 @@
             <material name="white"/>
         </visual>
+        <collision>
+            <origin xyz="0.15 0 0.075"/>
+            <geometry>
+                <box size="0.3 0.3 0.15"/>
+            </geometry>
+        </collision>
     </link>
     <!--LEFT WHEEL LINK-->
@@ -45,4 +51,9 @@
             <material name="blue"/>
         </visual>
+        <collision>
+            <geometry>
+                <cylinder radius="0.05" length="0.04"/>
+            </geometry>
+        </collision>
     </link>
     <!--RIGHT WHEEL LINK-->
@@ -60,4 +71,9 @@
             <material name="blue"/>
         </visual>
+        <collision>
+            <geometry>
+                <cylinder radius="0.05" length="0.04"/>
+            </geometry>
+        </collision>
     </link>
     <!--CASTER WHEEL-->
@@ -74,4 +90,9 @@
             <material name="black"/>
         </visual>
+        <collision>
+            <geometry>
+                <sphere radius="0.05" />
+            </geometry>
+        </collision>
     </link>
 </robot>

Commit message: inertia

File: description/robot_core.xacro (robot description, xacro)
@@ -1,4 +1,5 @@
 <?xml version="1.0"?>
 <robot xmlns:xacro="http://www.ros.org/wiki/xacro" >
+    <xacro:include filename="inertial_macros.xacro"/>
     <material name="white">
         <color rgba="1 1 1 1" />
@@ -36,4 +37,6 @@
             </geometry>
         </collision>
+        <xacro:inertial_box mass="0.5" x="0.3" y="0.3" z="0.15" />
+            <origin xyz="0.15 0 0.075"/>
     </link>
     <!--LEFT WHEEL LINK-->
@@ -56,4 +59,7 @@
             </geometry>
         </collision>
+        <xacro:inertial_cylinder mass="0.1" length="0.04" radius="0.05" />
+            <origin xyz="0 0 0" rpy="0 0 0"/>
+        </xacro:inertial_cylinder>
     </link>
     <!--RIGHT WHEEL LINK-->
@@ -76,4 +82,7 @@
             </geometry>
         </collision>
+        <xacro:inertial_cylinder mass="0.1" length="0.04" radius="0.05" />
+            <origin xyz="0 0 0" rpy="0 0 0"/>
+        </xacro:inertial_cylinder>
     </link>
     <!--CASTER WHEEL-->
@@ -95,4 +104,7 @@
             </geometry>
         </collision>
+        <xacro:inertial_sphere mass="0.1" radius="0.05" />
+            <origin xyz="0 0 0"/>
+        </xacro:inertial_sphere>
     </link>
 </robot>

Commit message: colors

File: description/robot_core.xacro (robot description, xacro)
@@ -41,4 +41,7 @@
         </xacro:inertial_box>
     </link>
+    <gazebo reference="chassis">
+        <material>Gazebo/White</material>
+    </gazebo>
     <!--LEFT WHEEL LINK-->
     <joint name="left_wheel_joint" type="continuous">
@@ -64,4 +67,7 @@
         </xacro:inertial_cylinder>
     </link>
+    <gazebo reference="left_wheel">
+        <material>Gazebo/blue</material>
+    </gazebo>
     <!--RIGHT WHEEL LINK-->
     <joint name="right_wheel_joint" type="continuous">
@@ -87,4 +93,7 @@
         </xacro:inertial_cylinder>
     </link>
+    <gazebo reference="right_wheel">
+        <material>Gazebo/blue</material>
+    </gazebo>
     <!--CASTER WHEEL-->
     <joint name="caster_wheel_joint" type="fixed">
@@ -109,3 +118,6 @@
         </xacro:inertial_sphere>
     </link>
+    <gazebo reference="caster_wheel">
+        <material>Gazebo/black</material>
+    </gazebo>
 </robot>

Commit message: color change error

File: description/robot_core.xacro (robot description, xacro)
@@ -68,5 +68,5 @@
     </link>
     <gazebo reference="left_wheel">
-        <material>Gazebo/blue</material>
+        <material>Gazebo/Blue</material>
     </gazebo>
     <!--RIGHT WHEEL LINK-->
@@ -94,5 +94,5 @@
     </link>
     <gazebo reference="right_wheel">
-        <material>Gazebo/blue</material>
+        <material>Gazebo/Blue</material>
     </gazebo>
     <!--CASTER WHEEL-->
@@ -119,5 +119,5 @@
     </link>
     <gazebo reference="caster_wheel">
-        <material>Gazebo/black</material>
+        <material>Gazebo/Black</material>
     </gazebo>
 </robot>
