Commit message: link and base editing

File: description/robot.urdf.xacro (robot description, xacro)
@@ -1,6 +1,4 @@
 <?xml version="1.0"?>
-<robot xmlns:xacro="http://www.ros.org/wiki/xacro"  name="robot">
-    <!-- Example link -->
-    <link name="base_link"></link>
-    <xacro:include filename="robot_core.xacro">
+<robot xmlns:xacro="http://www.ros.org/wiki/xacro" name="robot">
+    <xacro:include filename="robot_core.xacro" />
 </robot>

File: description/robot_core.xacro (robot description, xacro)
@@ -13,10 +13,10 @@
         <color rgba="0 0 0 1" />
     </material>
-    <link name=base_link>
+    <link name="base_link">
     </link>
     <joint name="chassis_joint" type="fixed">
         <parent link="base_link"/>
         <child link="chassis"/>
-        <origin xyz="-.1 0 0"/>
+        <origin xyz="-0.1 0 0"/>
     </joint>
     <link name="chassis">
@@ -26,5 +26,5 @@
                 <box size="0.3 0.3 0.15"/>
             </geometry>
-            <material name="white">
+            <material name="white"/>
         </visual>
     </link>

Commit message: lidar

File: description/robot.urdf.xacro (robot description, xacro)
@@ -3,3 +3,4 @@
     <xacro:include filename="robot_core.xacro" />
     <xacro:include filename="gazebo_control.xacro"/>
+    <xacro:include filename="lidar.xacro"/>
 </robot>

File: description/robot_core.xacro (robot description, xacro)
@@ -13,4 +13,7 @@
     <material name="black">
         <color rgba="0 0 0 1" />
+    </material>
+    <material name="red">
+        <color rgba="1 0 0 1" />
     </material>
     <!--BASE LINK-->
